File: Hardware/module_version/Analog.kicad_sch (KiCad schematic)
At the start: 20 parts

Commit message: work in progress...
Parts:
- added JP1, JP2, JP3, JP4: Jumper_2_Open, Jumper:SolderJumper-2_P1.3mm_Open_RoundedPad1.0x1.5mm, symbol Jumper:Jumper_2_Open
- C10, C11, C12, C13: value 100n -> 100n 16V; footprint Capacitor_SMD:C_0603_1608Metric -> Capacitor_SMD:C_0402_1005Metric; symbol RoboPonteDual-rescue:C -> Device:C; LCSC C14663 -> C60474; MFR (none) -> CC0402KRX7R7BB104; katodo 10.1050.0004 -> (none)
- P1, P2, P3, P4: symbol RoboPonteDual-rescue:CONN_01X02 -> Connector_Generic:Conn_01x02
- R21, R22, R29, R30: value 10K -> 1K87; symbol RoboPonteDual-rescue:R -> Device:R; LCSC C25804 -> C843924; MFR (none) -> CRCW06031K87FKEA
- R23, R24, R31, R32: symbol RoboPonteDual-rescue:R -> Device:R
Connections:
- net GND: now also JP1.2 (B), JP2.2 (B), JP3.2 (B), JP4.2 (B); no longer R21.2, R22.2, R29.2, R30.2
- net I1: now reaches P1.2 (Pin_2), R23.1
- net V1: now reaches P3.2 (Pin_2), R31.1
- net V2: now reaches P4.2 (Pin_2), R32.1
- net I2: now reaches P2.2 (Pin_2), R24.1
- new net: JP1.1 (A), R21.2
- new net: JP4.1 (A), R30.2
- new net: JP3.1 (A), R22.2
- new net: JP2.1 (A), R29.2
Other:
- note added: "OPEN: 3V3 input CLOSED: 5V1 input"
- note added: "hBridge3620 -> CLOSED"
- note added: "hBridge3620 -> OPEN"
- company: Katodo di Mauro Soligo -> Mauro Soligo
- moved on the sheet: C10, C11, C12, C13, D6, D7, D8, D9, R21, R22, R23, R24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
