File: Hardware/module_version/RobotMotorController.kicad_sch (KiCad schematic)
At the start: 12 parts, among them J3 CONN_01x04, J4 CONN_01x04, J5 CONN_01x04, J9 CONN_01x04, U1 RP2040-rgb

Commit message: Work in progress on rm2040 module version.
Parts:
- added C30 (x5): 100n 50V Y5V, Capacitor_SMD:C_0402_1005Metric, symbol Device:C
- added R44 (x6): 0Ω/S4, Resistor_SMD:R_0402_1005Metric, symbol Device:R
- added R44 (x2): 1K/S4, Resistor_SMD:R_0402_1005Metric, symbol Device:R
- added U5: ADS1115IDGS, Package_SO:TSSOP-10_3x3mm_P0.5mm, symbol Analog_ADC:ADS1115IDGS
- added U7: INA3221, Package_DFN_QFN:Texas_RGV_S-PVQFN-N16_EP2.1x2.1mm, symbol Power_Management:INA3221
- TP52: footprint TestPoint:TestPoint_Pad_D2.0mm -> TestPoint:TestPoint_THTPad_D2.5mm_Drill1.2mm
Connections:
- net +3V3: now also C30.2, C30.2, R44.1, R44.1, R44.2, R44.2, U5.8 (VDD), U7.4 (VS)
- net GND: now also C30.1, C30.1, U5.3 (GND), U7.17 (EP), U7.3 (GND)
- new net: R44.1, R44.1, R44.1, U7.5 (A0)
- new net: R44.1, R44.1, R44.1, U5.1 (ADDR)
- new net A0_VBUS: U5.4 (AIN0)
- new net A1_VJETSON: U5.5 (AIN1)
- new net A2_VBATT: U5.6 (AIN2)
- new net A3_BATT_T: U5.7 (AIN3)
- new net IB_n: C30.1, U7.14 (IN-2)
- new net IB_p: C30.2, U7.15 (IN+2)
- new net IJ_n: C30.1, U7.1 (IN-3)
- new net IJ_p: C30.2, U7.2 (IN+3)
- new net IS_n: C30.1, U7.11 (IN-1)
- new net IS_p: C30.2, U7.12 (IN+1)
- new net SCL2: R44.2, R44.2, R44.2, U5.10 (SCL), U7.6 (SCL)
- new net SDA2: R44.2, R44.2, R44.2, U5.9 (SDA), U7.7 (SDA)
Other:
- note added: "0x41"
- note added: "0x42"
- note added: "0x43"
- note added: "0x49"
- note added: "0x4A"
- note added: "0x4B"
- note added: "A0 - SLAVE ADDR GND - 1000000 0x40 VS - 1000001 0x41 SDA - 1000010 0x42 SCL - 1000011 0x43 In Jetson Nano there is another I2C device with address 0x40"
- note added: "A0 - SLAVE ADDR GND - 1001000 0x48 VS - 1001001 0x49 SDA - 1001010 0x4A SCL - 1001011 0x4B"
- note added: "CURRENT MONITOR"
- note added: "VOLTAGE MONITOR"

Commit message: work in progress...
Parts:
- removed C30 (x5): 100n 50V Y5V, Capacitor_SMD:C_0402_1005Metric, symbol Device:C
- removed R44 (x6): 0Ω/S4, Resistor_SMD:R_0402_1005Metric, symbol Device:R
- removed R44 (x2): 1K/S4, Resistor_SMD:R_0402_1005Metric, symbol Device:R
- removed TP52 (x3): TestPoint, TestPoint:TestPoint_THTPad_D2.5mm_Drill1.2mm, symbol Connector:TestPoint
- removed U5: ADS1115IDGS, Package_SO:TSSOP-10_3x3mm_P0.5mm, symbol Analog_ADC:ADS1115IDGS
- removed U7: INA3221, Package_DFN_QFN:Texas_RGV_S-PVQFN-N16_EP2.1x2.1mm, symbol Power_Management:INA3221
- added JP2: Jumper_2_Open, Jumper:SolderJumper-2_P1.3mm_Open_RoundedPad1.0x1.5mm, symbol Jumper:Jumper_2_Open
- added R44 (x2): 1K/S4, Resistor_SMD:R_0402_1005Metric, symbol Device:R
- J3, J4, J5, J9: symbol agg-kicad:CONN_01x04 -> Connector_Generic:Conn_01x04; now in the parts list
Connections:
- net +3V3: now also R44.1, R44.1; no longer U1.41 (3V3)
- net GND: no longer U1.44 (GND)
- net I2C0-SCL: now also R44.2
- net I2C0-SDA: now also R44.2
- net I2C0-ALERT: now reaches U1.29 (GP22)
- net at U1.39 (VIN): now also JP2.1 (A)
- net SWCLK: no longer names the net of U1.43 (SWCLK)
- net SWD: no longer names the net of U1.42 (SWDIO)
- new net +5V: JP2.2 (B)
- no-connect marks 2 -> 10
Other:
- added sheet PowerOut (powerout.kicad_sch)
- sheet Supply and Power ports: added I2C0-ALERT, I2C0-SCL, I2C0-SDA; removed none
- note added: "For SWD use, connect directly on the module."
- note removed: "0x41"
- note removed: "0x42"
- note removed: "0x43"
- note removed: "0x49"
- note removed: "0x4A"
- note removed: "0x4B"
- note removed: "A0 - SLAVE ADDR GND - 1000000 0x40 VS - 1000001 0x41 SDA - 1000010 0x42 SCL - 1000011 0x43 In Jetson Nano there is another I2C device with address 0x40"
- note removed: "A0 - SLAVE ADDR GND - 1001000 0x48 VS - 1001001 0x49 SDA - 1001010 0x4A SCL - 1001011 0x4B"
- note removed: "CURRENT MONITOR"
- note removed: "VOLTAGE MONITOR"
- company: Katodo di Mauro Soligo -> Mauro Soligo
- moved on the sheet: U1
