File: Hardware/module_version/motor.kicad_sch (KiCad schematic)
At the start: 24 parts

Commit message: work in progress...
Parts:
- C1, C14, C15, C2: value 100n -> 100n 16V; footprint Capacitor_SMD:C_0603_1608Metric -> Capacitor_SMD:C_0402_1005Metric; symbol MotorController:SPARKFUN-CAPACITORS_CAP -> Device:C; KATODO 10.1050.0023 -> (none); LCSC C14663 -> C60474; MFR (none) -> CC0402KRX7R7BB104
- E1, E2: symbol RoboPonteDual-rescue:CONN_01X05 -> Connector_Generic:Conn_01x05
- M1, M2: symbol RoboPonteDual-rescue:CONN_01X06 -> Connector_Generic:Conn_01x06; now in the parts list
- R1, R10, R11, R12, R13, R14, R15, R18, R2, R20, R3, R4, R5, R7, R8, R9: symbol RoboPonteDual-rescue:R -> Device:R
Connections:
- net E1_CHA: no longer E1.2 (P2), R4.1
- net E1_CHB: no longer E1.3 (P3), R5.1
- net E2_CHA: no longer E2.2 (P2), R1.1
- net E2_CHB: no longer E2.3 (P3), R2.1
- new net E1_CHA_OUT: E1.2 (Pin_2), R4.1
- new net E1_CHB_OUT: E1.3 (Pin_3), R5.1
- new net E2_CHA_OUT: E2.2 (Pin_2), R1.1
- new net E2_CHB_OUT: E2.3 (Pin_3), R2.1
- no-connect marks 0 -> 2
Other:
- company: Katodo di Mauro Soligo -> Mauro Soligo
