File: Hardware/module_version/motor.kicad_sch (KiCad schematic)
At the start: 24 parts

Commit message: Final version - Production 22/01/2024
Parts:
- R15, R18, R20, R3: LCSC C4190 -> C227664
Changed lines of the file:
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@@
       (effects (font (size 1.27 1.27)))
     )
-    (property "LCSC" "C4190" (at 132.08 48.26 0)
+    (property "LCSC" "C227664" (at 132.08 48.26 0)
       (effects (font (size 1.27 1.27)) hide)
     )
@@
       (effects (font (size 1.27 1.27)))
     )
-    (property "LCSC" "C4190" (at 132.08 33.02 0)
+    (property "LCSC" "C227664" (at 132.08 33.02 0)
       (effects (font (size 1.27 1.27)) hide)
     )
@@
       (effects (font (size 1.27 1.27)))
     )
-    (property "LCSC" "C4190" (at 132.08 27.94 0)
+    (property "LCSC" "C227664" (at 132.08 27.94 0)
       (effects (font (size 1.27 1.27)) hide)
     )
@@
       (effects (font (size 1.27 1.27)))
     )
-    (property "LCSC" "C4190" (at 132.08 43.18 0)
-      (effects (font (size 1.27 1.27)) hide)
-    )
+    (property "LCSC" "C227664" (at 132.08 43.18 0)
+      (effects (font (size 1.27 1.27)) hide)
+    )
