File: Hardware/module_version/powerout.kicad_sch (KiCad schematic)
At the start: 16 parts, among them J8 XT60PW-M, U4 INA237, U5 INA237

Commit message: Rev 0.9, ready to check...
Connections:
- net GND: now also J8.1 (-), J8.1 (-); no longer J8.2 (-), J8.2 (-)
- net at R44.1, R44.2: now also J8.2 (+); no longer J8.1 (+) (x2)
