File: Hardware/module_version/supply.kicad_sch (KiCad schematic)
At the start: 21 parts, among them J21 Power Input, U32 TLV1117LV33DCYR, U33 TX4139

Commit message: work in progress...
Parts:
- added C10 (x2): 100n 16V, Capacitor_SMD:C_0402_1005Metric, symbol Device:C
- added NT3: NetTie_2, NetTie:NetTie-2_SMD_Pad0.5mm, symbol Device:NetTie_2
- added R44: 10mΩ 2W, Resistor_SMD:R_2512_6332Metric_Pad1.40x3.35mm_HandSolder, symbol Device:R
- added R44 (x2): 10Ω/S4, Resistor_SMD:R_0402_1005Metric, symbol Device:R
- added U5: INA237, Package_SO:VSSOP-10_3x3mm_P0.5mm, symbol katodo_kicad:INA237
- C114: value 100n -> 100n 16V; footprint Capacitor_SMD:C_0603_1608Metric -> Capacitor_SMD:C_0402_1005Metric; LCSC C14663 -> C60474; MFR (none) -> CC0402KRX7R7BB104
- R98: footprint Resistor_SMD:R_0603_1608Metric -> Resistor_SMD:R_0402_1005Metric_Pad0.72x0.64mm_HandSolder; LCSC C22859 -> C138066
- U32: symbol Regulator_Linear:NCP1117-3.3_SOT223 -> katodo_kicad:NCP1117-3.3_SOT223
- U33: symbol MotorBuck:TX4139 -> katodo_kicad:TX4139
Connections:
- net +3V3: now also TP52.1, C10.1, U5.6 (VS); no longer TP52.1
- net GND: now also TP52.1, C10.2, U5.1 (A1), U5.2 (A0), U5.7 (GND); no longer TP52.1
- net Vdrive: now also NT3.2, R44.2, R44.2
- new net: C10.2, R44.1, U5.10 (IN+)
- new net: NT3.1, U5.8 (VBUS)
- new net: C10.1, R44.1, U5.9 (IN-)
- new net BATT_OUT: R44.1, R44.2
- new net I2C0-ALERT: U5.3 (ALERT)
- new net I2C0-SCL: U5.5 (SCL)
- new net I2C0-SDA: U5.4 (SDA)
- no-connect marks 0 -> 2
Other:
- note added: "10mΩ @ 30A = 0.9W"
- note added: "A1 A0 SEC. ADDRESS AVAILABLE GND GND 1000000 64 (MAIN) GND VS 1000001 65 (MOTOR1) GND SDA 1000010 66 (MOTOR2) GND SCL 1000011 VS GND 1000100 VS VS 1000101 VS SDA 1000110 VS SCL 1000111 SDA GND 1001000 SDA VS 1001001 SDA SDA 1001010 SDA SCL 1001011 SCL GND 1001100 SCL VS 1001101 SCL SDA 1001110 SCL SCL 1001111"
- company: Katodo di Mauro Soligo -> Mauro Soligo
- moved on the sheet: C110, C111, C112, C113, C114, C115, C122, C26, D27, D4, J21, L3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

Commit message: Rev 0.9, ready to check...
Parts:
- removed J21: Power Input, Connector_AMASS:AMASS_XT60-F_1x02_P7.20mm_Vertical, symbol Connector_Generic:Conn_01x02
- added J1: XT60PW-F, Connector_AMASS:AMASS_XT60-F_1x02_P7.20mm_Vertical, symbol katodo_kicad:XT60PW-F
- C26: value 47uF 63V solid -> 47uF 50V; footprint Capacitor_THT:CP_Radial_D8.0mm_P3.50mm -> Capacitor_THT:CP_Radial_D8.0mm_P5.00mm
Connections:
- net GND: now also J1.1 (-)
- net Vdrive: now also J1.2 (+)
Changed lines of the file:
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@@
       (effects (font (size 1.778 1.778)) (justify bottom))
     )
-    (property "Value" "47uF 63V solid" (at 63.5 129.54 90)
+    (property "Value" "47uF 50V" (at 63.5 129.54 90)
       (effects (font (size 1.651 1.651)) (justify top))
     )
-    (property "Footprint" "Capacitor_THT:CP_Radial_D8.0mm_P3.50mm" (at 69.5452 133.35 0)
+    (property "Footprint" "Capacitor_THT:CP_Radial_D8.0mm_P5.00mm" (at 69.5452 133.35 0)
       (effects (font (size 1.27 1.27)) hide)
     )
@@
     )
   )
-  (symbol (lib_id "Connector_Generic:Conn_01x02") (at 106.68 30.48 0) (mirror y) (unit 1)
-    (in_bom no) (on_board yes) (dnp no)
-    (property "Reference" "J21" (at 104.14 30.48 0)
-      (effects (font (size 1.27 1.27)) (justify left))
-    )
-    (property "Value" "Power Input" (at 104.14 31.75 0)
-      (effects (font (size 1.27 1.27)) (justify left))
-    )
-    (property "Footprint" "Connector_AMASS:AMASS_XT60-F_1x02_P7.20mm_Vertical" (at 106.68 30.48 0)
-      (effects (font (size 1.27 1.27)) hide)
-    )
-    (property "Datasheet" "~" (at 106.68 30.48 0)
-      (effects (font (size 1.27 1.27)) hide)
-    )
-    (pin "1")
-    (pin "2")
-    (instances
-      (project "RP2040_motor"
-        (path "/10ff4ace-8dac-45ce-94a5-ae8ae7d42914/11bddbd5-e14e-4409-876e-6e46bce03704"
-          (reference "J21") (unit 1)
-        )
-      )
-      (project "power_and_cpu"
-        (path "/8d16b105-3293-4d6d-a54b-7359568d7527"
-          (reference "J21") (unit 1)
-        )
-      )
-      (project "RobotMotorController"
-        (path "/e63e39d7-6ac0-4ffd-8aa3-1841a4541b55"
-          (reference "J27") (unit 1)
-        )
-        (path "/e63e39d7-6ac0-4ffd-8aa3-1841a4541b55/4b47efe4-f44f-4b9c-acfc-3b1272cbd0ae"
-          (reference "J1") (unit 1)
-        )
-      )
-    )
-  )
   (symbol (lib_id "power:GND") (at 152.4 71.12 270) (unit 1)
     (in_bom yes) (on_board yes) (dnp no) (fields_autoplaced)
@@
         )
       )
+    )
+  )
+  (symbol (lib_id "katodo_kicad:XT60PW-F") (at 101.6 33.02 0) (mirror y) (unit 1)
+    (in_bom yes) (on_board yes) (dnp no) (fields_autoplaced)
+    (property "Reference" "J1" (at 101.6 22.86 0)
+      (effects (font (size 1.27 1.27)))
+    )
+    (property "Value" "XT60PW-F" (at 101.6 25.4 0)
+      (effects (font (size 1.27 1.27)))
+    )
+    (property "Footprint" "Connector_AMASS:AMASS_XT60-F_1x02_P7.20mm_Vertical" (at 101.6 33.02 0)
+      (effects (font (size 1.27 1.27)) (justify bottom) hide)
+    )
+    (property "Datasheet" "" (at 101.6 33.02 0)
+      (effects (font (size 1.27 1.27)) hide)
+    )
+    (property "PARTREV" "V1.2" (at 101.6 33.02 0)
+      (effects (font (size 1.27 1.27)) (justify bottom) hide)
+    )
+    (property "MANUFACTURER" "AMASS" (at 101.6 33.02 0)
+      (effects (font (size 1.27 1.27)) (justify bottom) hide)
+    )
+    (property "MAXIMUM_PACKAGE_HEIGHT" "8.4 mm" (at 101.6 33.02 0)
+      (effects (font (size 1.27 1.27)) (justify bottom) hide)
+    )
+    (property "STANDARD" "Manufacturer recommendations" (at 101.6 33.02 0)
+      (effects (font (size 1.27 1.27)) (justify bottom) hide)
+    )
+    (property "Description" "~" (at 101.6 33.02 0)
+      (effects (font (size 1.27 1.27)) hide)
+    )
+    (property "LCSC" "~" (at 101.6 33.02 0)
+      (effects (font (size 1.27 1.27)) hide)
+    )
+    (pin "2")
+    (pin "1")
+    (instances
+      (project "RobotMotorController"
+        (path "/e63e39d7-6ac0-4ffd-8aa3-1841a4541b55/4b47efe4-f44f-4b9c-acfc-3b1272cbd0ae"
+          (reference "J1") (unit 1)
+        )
+      )
