File: Hardware/module_version/RobotMotorController.kicad_pcb (KiCad board)
At the start: 2 copper layers, 80 x 85 mm, 148 parts, among them J1 Power Input, J2 Conn_01x05, J5 CONN_01x04, J9 CONN_01x04, Q2 BSS138, Q3 BSS138, Q4 BSS138, U1 RP2040-rgb, U10 TX4139, U3 #DS18B20, U8 TLV1117LV33DCYR

Commit message: Work in progress on rm2040 module version.
Parts:
- removed C16: 100n, Capacitor_SMD:C_0603_1608Metric
- removed D11, D12, D13: 1N4148W, Diode_SMD:D_SOD-123
- removed J2: Conn_01x05, Katodo:DG300-5.0-05P-13
- removed Q2, Q3, Q4: BSS138, Package_TO_SOT_SMD:SOT-23
- removed R17, R19: 1K, Resistor_SMD:R_0603_1608Metric
- removed R34, R38, R40: 100R, Resistor_SMD:R_0603_1608Metric
- removed R35, R37, R39, R41: 10K, Resistor_SMD:R_0603_1608Metric
- removed R36: 100K, Resistor_SMD:R_0603_1608Metric
- removed TP5, TP6, TP7, TP8: TESTPAD, TestPoint:TestPoint_Loop_D2.50mm_Drill1.85mm
- removed U3: #DS18B20, Package_TO_SOT_THT:TO-92_Inline
- removed kibuzzard-654DD07D: G***, kibuzzard-654DD07D
- added J3: CONN_01x04, Connector_Molex:Molex_KK-254_AE-6410-04A_1x04_P2.54mm_Vertical, F.Cu at (242.8, 171.6)
- added J4: CONN_01x04, Connector_Molex:Molex_KK-254_AE-6410-04A_1x04_P2.54mm_Vertical, F.Cu at (239.7, 107.6)
- added kibuzzard-654DCFB0: G***, kibuzzard-654DCFB0, F.Cu at (176.5, 164.0)
- added kibuzzard-654DCFBA: G***, kibuzzard-654DCFBA, F.Cu at (176.5, 166.6)
- added kibuzzard-654DCFC5: G***, kibuzzard-654DCFC5, F.Cu at (176.5, 169.1)
- added kibuzzard-654DCFCD: G***, kibuzzard-654DCFCD, F.Cu at (176.5, 171.6)
- TP1, TP2, TP3: footprint TestPoint:TestPoint_Pad_D2.0mm -> TestPoint:TestPoint_THTPad_D2.5mm_Drill1.2mm
- moved G*** 166.1 mm to (107.7, -22.9)
- moved TP1 154.4 mm to (197.6, 180.3)
- moved TP2 154.4 mm to (190.6, 180.3)
- moved TP3 154.4 mm to (194.1, 180.3)
- moved C1 152.0 mm to (238.3, 142.5), turned to 90 degrees
- moved kibuzzard-653F53EC 122.6 mm to (227.5, 101.0), turned to -90 degrees
- moved kibuzzard-654DCF33 120.0 mm to (225.0, 101.0), turned to -90 degrees
- moved kibuzzard-654DCF3E 117.3 mm to (222.4, 101.0), turned to -90 degrees
- moved J9 116.7 mm to (227.5, 107.6), turned to 180 degrees
- moved kibuzzard-654DCF59 114.7 mm to (219.9, 101.0), turned to -90 degrees
- moved kibuzzard-653F53F2 100.9 mm to (176.5, 158.9)
- moved C15 100.8 mm to (167.5, 167.3)
- moved C33 100.8 mm to (208.9, 107.5)
- moved E2 100.8 mm to (242.8, 158.9)
- moved H3 100.8 mm to (247.8, 177.8)
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Connections:
- net I2C-SCL renamed I2C0-SCL
- net I2C-SDA renamed I2C0-SDA
- net UART_RX renamed UART0_RX
- net UART_TX renamed UART0_TX
- U1 pad 11: MOT1_AUX -> UART1_TX
- U1 pad 12: MOT1_EN -> UART1_RX
- U1 pad 16: unconnected-(U1-GP12-Pad16) -> MOT1_AUX
- U1 pad 17: PWR_MOT_EN -> MOT1_EN
- U1 pad 19: PWR_SBC_EN -> unconnected-(U1-GP14-Pad19)
- U1 pad 20: PWR-REG-EN -> unconnected-(U1-GP15-Pad20)
- U1 pad 24: unconnected-(U1-GP18-Pad24) -> I2C1-SDA
- U1 pad 25: I2C-INT -> I2C1-SCL
- U1 pad 37: LED_DATA -> unconnected-(U1-GP23-Pad37)
Other:
- board text removed: "3V"
- board text removed: "DQ"
- board text removed: "G"

Commit message: work in progress...
Parts:
- removed TP1, TP2, TP3: TestPoint, TestPoint:TestPoint_THTPad_D2.5mm_Drill1.2mm
- added C18: 100n 16V, Capacitor_SMD:C_0402_1005Metric, F.Cu at (194.1, 137.0)
- added C3: 100n 16V, Capacitor_SMD:C_0402_1005Metric, F.Cu at (197.4, 116.5)
- added C4: 100n 16V, Capacitor_SMD:C_0402_1005Metric, F.Cu at (192.3, 118.6)
- added C5: 100n 16V, Capacitor_SMD:C_0402_1005Metric, F.Cu at (200.7, 122.9)
- added C6: 100n 16V, Capacitor_SMD:C_0402_1005Metric, F.Cu at (193.0, 132.9)
- added C9: 100n 16V, Capacitor_SMD:C_0402_1005Metric, F.Cu at (197.4, 121.0)
- added J10: XT60PW-M, Connector_AMASS:AMASS_XT60-M_1x02_P7.20mm_Vertical, F.Cu at (188.6, 178.1)
- added J8: XT60PW-M, Connector_AMASS:AMASS_XT60-M_1x02_P7.20mm_Vertical, F.Cu at (237.0, 178.1)
- added JP1: Jumper_2_Open, Jumper:SolderJumper-2_P1.3mm_Open_RoundedPad1.0x1.5mm, F.Cu at (214.6, 152.7)
- added JP2: Jumper_2_Open, Jumper:SolderJumper-2_P1.3mm_Open_RoundedPad1.0x1.5mm, F.Cu at (214.6, 160.0)
- added JP3: Jumper_2_Open, Jumper:SolderJumper-2_P1.3mm_Open_RoundedPad1.0x1.5mm, F.Cu at (214.6, 156.5)
- added JP4: Jumper_2_Open, Jumper:SolderJumper-2_P1.3mm_Open_RoundedPad1.0x1.5mm, F.Cu at (214.6, 163.6)
- added JP5: Jumper_2_Open, Jumper:SolderJumper-2_P1.3mm_Open_RoundedPad1.0x1.5mm, F.Cu at (207.3, 177.3)
- added NT1: NetTie_2, NetTie:NetTie-2_SMD_Pad0.5mm, F.Cu at (191.7, 129.9)
- added NT2: NetTie_2, NetTie:NetTie-2_SMD_Pad0.5mm, F.Cu at (197.2, 123.5)
- added NT3: NetTie_2, NetTie:NetTie-2_SMD_Pad0.5mm, F.Cu at (191.5, 115.2)
- added R16: 1K/S4, Resistor_SMD:R_0402_1005Metric, F.Cu at (206.3, 146.9)
- added R17: 10Ω/S4, Resistor_SMD:R_0402_1005Metric, F.Cu at (192.3, 116.6)
- added R19: 10Ω/S4, Resistor_SMD:R_0402_1005Metric, F.Cu at (192.3, 120.7)
- added R25: 10mΩ 2W, Resistor_SMD:R_2512_6332Metric_Pad1.40x3.35mm_HandSolder, F.Cu at (189.5, 118.4)
- added R36: 10Ω/S4, Resistor_SMD:R_0402_1005Metric, F.Cu at (192.5, 131.4)
- added R37: 10Ω/S4, Resistor_SMD:R_0402_1005Metric, F.Cu at (192.5, 134.5)
- added R38: 10mΩ 2W, Resistor_SMD:R_2512_6332Metric_Pad1.40x3.35mm_HandSolder, F.Cu at (189.5, 133.0)
- added R42: 10Ω/S4, Resistor_SMD:R_0402_1005Metric, F.Cu at (198.7, 122.9)
- added R44: 10Ω/S4, Resistor_SMD:R_0402_1005Metric, F.Cu at (202.8, 122.9)
- added R50: 10mΩ 2W, Resistor_SMD:R_2512_6332Metric_Pad1.40x3.35mm_HandSolder, F.Cu at (200.2, 125.6)
- added R6: 1K/S4, Resistor_SMD:R_0402_1005Metric, F.Cu at (206.3, 144.3)
- added U2: INA237, Package_SO:VSSOP-10_3x3mm_P0.5mm, F.Cu at (194.9, 118.8)
- added U4: INA237, Package_SO:VSSOP-10_3x3mm_P0.5mm, F.Cu at (199.8, 118.8)
- added U5: INA237, Package_SO:VSSOP-10_3x3mm_P0.5mm, F.Cu at (195.6, 133.0)
- added kibuzzard-653F53EC: G***, kibuzzard-653F53EC, F.Cu at (239.7, 101.0)
- added kibuzzard-654DCF33: G***, kibuzzard-654DCF33, F.Cu at (237.1, 101.0)
- added kibuzzard-654DCF3E: G***, kibuzzard-654DCF3E, F.Cu at (234.6, 101.0)
- added kibuzzard-654DCF59: G***, kibuzzard-654DCF59, F.Cu at (232.1, 101.0)
- added kibuzzard-655CCB55: G***, kibuzzard-655CCB55, F.Cu at (176.0, 161.5)
- added kibuzzard-655CCBF1: G***, kibuzzard-655CCBF1, F.Cu at (249.6, 161.5)
- C1, C10, C11, C12, C13, C14, C15, C2, C33: value 100n -> 100n 16V; footprint Capacitor_SMD:C_0603_1608Metric -> Capacitor_SMD:C_0402_1005Metric
- R21, R22, R29, R30: value 10K -> 1K87
- R45: footprint Resistor_SMD:R_0603_1608Metric -> Resistor_SMD:R_0402_1005Metric_Pad0.72x0.64mm_HandSolder
- moved C15 76.0 mm to (243.3, 161.5)
- moved TP14 58.3 mm to (258.1, 129.0)
- moved TP4 57.0 mm to (257.4, 124.1)
- moved TP15 46.8 mm to (256.4, 120.3)
- moved C20 42.6 mm to (164.0, 87.9), turned to -90 degrees
- moved C2 21.8 mm to (182.3, 146.3), turned to 180 degrees
- moved C19 21.5 mm to (210.5, 137.9), turned to 90 degrees
- moved C29 21.4 mm to (212.8, 137.6), turned to 90 degrees
- moved U8 21.4 mm to (212.8, 144.4)
- moved C14 15.2 mm to (182.4, 161.5), turned to 180 degrees
- moved R10 14.9 mm to (218.9, 141.8), turned to 0 degrees
- moved R9 14.9 mm to (218.9, 139.2)
- moved R5 7.91 mm to (218.9, 176.6)
- moved R1 7.90 mm to (218.9, 172.9)
- moved R2 7.87 mm to (218.9, 169.7)
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Connections:
- net Net-(P1-P2) renamed /Analog/I1
- net Net-(P2-P2) renamed /Analog/I2
- net Net-(P3-P2) renamed /Analog/V1
- net Net-(P4-P2) renamed /Analog/V2
- E1 pad 2: E1_CHA -> E1_CHA_OUT
- E1 pad 3: E1_CHB -> E1_CHB_OUT
- E2 pad 2: E2_CHA -> E2_CHA_OUT
- E2 pad 3: E2_CHB -> E2_CHB_OUT
- R1 pad 1: E2_CHA -> E2_CHA_OUT
- R2 pad 1: E2_CHB -> E2_CHB_OUT
- R21 pad 2: GND -> Net-(JP1-A)
- R22 pad 2: GND -> Net-(JP3-A)
- R29 pad 2: GND -> Net-(JP2-A)
- R30 pad 2: GND -> Net-(JP4-A)
- R4 pad 1: E1_CHA -> E1_CHA_OUT
- R5 pad 1: E1_CHB -> E1_CHB_OUT
- TP15 pad 1: +3V3 -> GND
- TP4 pad 1: GND -> +3V3
- U1 pad 29: unconnected-(U1-GP22-Pad29) -> I2C0-ALERT
- U1 pad 39: unconnected-(U1-VIN-Pad39) -> Net-(JP5-A)
- U1 pad 41: +3V3 -> unconnected-(U1-3V3-Pad41)
- U1 pad 42: /SWD -> unconnected-(U1-SWDIO-Pad42)
- U1 pad 43: /SWCLK -> unconnected-(U1-SWCLK-Pad43)
- U1 pad 44: GND -> unconnected-(U1-GND-Pad44)
Routing:
- net +3V3: track 0.00 -> 268.7 mm, vias 0 -> 6
- net GND: track 28.1 -> 219.5 mm, vias 0 -> 31
- net +5V: track 0.00 -> 178.5 mm, vias 0 -> 2
- net /Analog/V2: track 0.00 -> 89.6 mm, vias 0 -> 1
- net Net-(J8-+): track 0.00 -> 84.1 mm
- net /Analog/I2: track 0.00 -> 83.3 mm, vias 0 -> 1
- net PWMA1: track 0.00 -> 70.2 mm, vias 0 -> 3
- net PWMB1: track 0.00 -> 68.0 mm, vias 0 -> 3
- net /Analog/V1: track 0.00 -> 64.2 mm, vias 0 -> 2
- net I2C1-SCL: track 0.00 -> 63.3 mm, vias 0 -> 2
- net I2C1-SDA: track 0.00 -> 63.1 mm, vias 0 -> 2
- net I2C0-SDA: track 0.00 -> 58.4 mm, vias 0 -> 5
- net I2C0-SCL: track 0.00 -> 53.6 mm, vias 0 -> 5
- net PWMA2: track 0.00 -> 53.4 mm, vias 0 -> 3
- net /Analog/I1: track 0.00 -> 52.9 mm, vias 0 -> 2
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- added copper zone on F.Cu, net +5V
- added copper zone on F.Cu, net /Supply and Power/SW
- added copper zone on F.Cu, net BATT_OUT
- added copper zone on F.Cu, net GND
- added copper zone on F.Cu, net Vdrive

Commit message: Rev 0.9, ready to check...
Parts:
- removed G***: LOGO, katodo:Katodo
- removed the kibuzzard-653D1AE4 at (155.0, -19.7)
- removed kibuzzard-653D1AEE: G***, kibuzzard-653D1AEE
- removed kibuzzard-653D1AF5: G***, kibuzzard-653D1AF5
- removed kibuzzard-653D1B0A: G***, kibuzzard-653D1B0A
- removed kibuzzard-653D1B23: G***, kibuzzard-653D1B23
- added kibuzzard-6576B604: G***, kibuzzard-6576B604, F.Cu at (223.7, 112.5)
- added kibuzzard-6576B615: G***, kibuzzard-6576B615, F.Cu at (235.9, 112.4)
- C20: value 47uF 63V solid -> 47uF 50V; footprint Capacitor_THT:CP_Radial_D8.0mm_P3.50mm -> Capacitor_THT:CP_Radial_D8.0mm_P5.00mm
- J1: value Power Input -> XT60PW-F
- moved TP14 45.7 mm to (214.3, 115.9), turned to 0 degrees
- moved TP4 39.6 mm to (218.7, 115.9)
- moved C20 35.3 mm to (187.8, 114.0), turned to 0 degrees
- moved TP15 32.4 mm to (224.4, 115.5)
- moved R24 10.5 mm to (198.7, 149.1), turned to -90 degrees
- moved R32 9.69 mm to (198.7, 157.5), turned to -90 degrees
- moved C18 8.66 mm to (197.3, 129.0)
- moved R23 8.06 mm to (200.4, 149.1), turned to -90 degrees
- moved R31 7.29 mm to (200.4, 157.5), turned to -90 degrees
- moved J10 7.20 mm to (195.8, 178.1), turned to 180 degrees
- moved J8 7.20 mm to (229.8, 178.1), turned to 0 degrees
- moved J1 7.20 mm to (196.0, 104.8), turned to 180 degrees
- moved D15 6.86 mm to (198.1, 113.7)
- moved C4 3.95 mm to (192.0, 122.5)
- moved R17 3.95 mm to (192.0, 120.5)
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Connections:
- J1 pad 1: Vdrive -> GND
- J1 pad 2: GND -> Vdrive
- J10 pad 1: Net-(J10-+) -> GND
- J10 pad 2: GND -> Net-(J10--)
- J8 pad 1: Net-(J8-+) -> GND
- J8 pad 2: GND -> Net-(J8-+)
- R37 pad 2: Net-(J10-+) -> Net-(J10--)
- R38 pad 1: Net-(J10-+) -> Net-(J10--)
Routing:
- net GND: track 219.5 -> 677.1 mm, vias 31 -> 60
- net +5V: track 178.5 -> 274.3 mm, vias 2 -> 8
- net UART1_TX: track 0.00 -> 51.4 mm, vias 0 -> 1
- net UART1_RX: track 0.00 -> 49.7 mm, vias 0 -> 1
- net UART0_RX: track 0.00 -> 46.3 mm, vias 0 -> 1
- net Net-(J10--): track 0.00 -> 46.2 mm
- net UART0_TX: track 0.00 -> 45.9 mm, vias 0 -> 1
- net Net-(J10-+): track 42.9 -> 0.00 mm
- net I2C0-ALERT: track 20.8 -> 50.3 mm, vias 4 -> 6
- net I2C0-SCL: track 53.6 -> 80.4 mm
- net +3V3: track 268.7 -> 242.2 mm, vias 6 -> 9
- net Vdrive: track 38.5 -> 63.7 mm
- net I2C0-SDA: track 58.4 -> 82.3 mm, vias 5 -> 7
- net /Analog/I2: track 83.3 -> 62.6 mm
- net /Analog/I1: track 52.9 -> 37.6 mm
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- added copper zone on B.Cu, net GND
Other:
- board text added: "RMC2040 1.0"
- board text removed: "3V3"
- board text removed: "5V"
- board text removed: "GND"
- board text removed: "pNav32 1.0"

Commit message: backup
Parts:
- R45: value 10Ω -> 10Ω/S4
Connections:
- net Net-(J10--) renamed /PowerOut/Vout2
- net Net-(J8-+) renamed /PowerOut/Vout1
Routing:
- net PWMB2: track 44.9 -> 45.5 mm
- net PWMA2: track 47.6 -> 48.1 mm
Other:
- board text added: "mauro.soligo@gmail.com"
